File: eagle/ESP8266.brd (EAGLE design)
At the start: 44.1 x 73.7 mm, 7 parts, among them IC1 LM2574HVM-3.3, U1 SN74AHCT125D

Commit message: board updated
Parts:
- added C1, C2: (no value), e-kondensatoren:GEPOLTER_ELEKTROLYTKONDENSATOR
- added L1: L1, e-spulen-transformatoren:SPULE
- moved JP2 23.3 mm to (12.7, 58.4), turned to 0 degrees
- moved U1 23.2 mm to (31.8, 53.3), turned to 90 degrees
- moved JP1 18.0 mm to (8.89, 44.5), flipped to the bottom, turned to 270 degrees
- moved D1 16.6 mm to (17.8, 68.6)
- moved R3 14.5 mm to (25.4, 76.2)
- moved WEMOS1 7.18 mm to (26.7, 27.9), turned to 0 degrees
- moved IC1 5.24 mm to (34.3, 66.0), turned to 0 degrees
Connections:
- removed net N$3: D1.2, IC1.12
- new net FB: C2.+, IC1.3, L1.2
- new net N$4: JP2.1
- new net OUT: D1.2, IC1.12, L1.1
- net 5V: now also C1.+
- net GND: now also C1.-, C2.-
- net N$1: no longer IC1.3, JP2.1
Routing:
- net N$1: track 44.4 -> 0.00 mm
- net 5V: track 86.5 -> 50.8 mm, vias 0 -> 1
- net SIGOUT(5V): track 8.82 -> 43.0 mm
- net GND: track 102.4 -> 133.7 mm, vias 0 -> 2
- net FB: track 0.00 -> 25.2 mm
- net OUT: track 0.00 -> 16.1 mm
- net N$3: track 16.0 -> 0.00 mm
- net DOUT: track 18.1 -> 29.4 mm, vias 0 -> 2
- net DIN: track 33.9 -> 24.4 mm
Other:
- board size 44.1 x 73.7 mm -> 44.1 x 80 mm

Commit message: great fileupdate
Parts:
- removed D1: (no value), diode:TO92H
- removed IC1: LM2574HVM-3.3, linear:SO14W
- removed JP2: (no value), jumper:JP2
- removed L1: L1, e-spulen-transformatoren:SPULE
- removed R3: 650k, eagle-ltspice:R0201
- added R1: (no value), eagle-ltspice:0204/7
- added U2: stepdown 5v to 3.3V, stepdown:STEPDOWN
- C1, C2: value (none) -> 100uF
- moved C2 26.1 mm to (16.5, 55.9)
- moved C1 19.4 mm to (30.5, 57.1)
- moved U1 16.6 mm to (33.0, 36.8), turned to 0 degrees
- moved WEMOS1 15.9 mm to (19.1, 14.0), turned to 90 degrees
- moved JP1 6.35 mm to (12.7, 39.4), flipped to the top, turned to 90 degrees
Connections:
- removed net FB: C2.+, IC1.3, L1.2
- removed net N$1: WEMOS1.3V3
- removed net N$4: JP2.1
- removed net OUT: D1.2, IC1.12, L1.1
- new net VOUT: C2.+, U2.VOUT, WEMOS1.3V3
- net 5V: now also U2.VIN; no longer IC1.10, JP2.3
- net DOUT: now also R1.2; no longer R3.2
- net GND: now also U2.GND; no longer D1.1, IC1.4, IC1.5, IC1.6, JP2.2
- net SIGOUT(5V): now also R1.1; no longer R3.1
Routing:
- net VOUT: track 0.00 -> 64.3 mm
- net GND: track 133.7 -> 72.9 mm, vias 2 -> 0
- net SIGOUT(5V): track 43.0 -> 2.70 mm
- net DOUT: track 29.4 -> 4.14 mm, vias 2 -> 0
- net FB: track 25.2 -> 0.00 mm
- net DIN: track 24.4 -> 45.7 mm
- net OUT: track 16.1 -> 0.00 mm
- net 5V: track 50.8 -> 60.1 mm, vias 1 -> 0
Other:
- board size 44.1 x 80 mm -> 46.7 x 80 mm
